Commit message: feat: surus kartinin 0x30 blogunu konus, freni kipe bagla, panolari ayir
Aracin kodu 31 Agustos'tan beri Mega'yi (/dev/mega @115200, 0x10-0x23)
bekliyordu; kart F767ZI'ye gecti ve 0x30-0x3E konusuyor. Ortusme sifir
oldugu icin /odom, /imu/data, /rc_input, seri E-STOP ve surus kipi
birden susuyordu. Bu commit o kopuklugu kapatiyor.

8 Eylul'de aracta olculdu: /dev/f767 @921600'de XOR'u tutan cerceve
geliyor ve uzun sure tek bozuk paket cikmiyor. Yani kablo, baud ve
cerceveleme dogruymus; konusamamanin tek sebebi bu koddu. Jetson->kart
yonu (0x39 JDR_LINK) hala kanitlanmadi.

KART ARAYUZU
- seri_kopru bastan yazildi: 0x30-0x3E cozumu, 0x01-0x09 gonderimi
- 0x09 ayar paketi; kart RAM'de tuttugu icin kalicilik koprude: kart
  ilk gorunduğunde ve her resetinde (0x35 v1 geri sarmasi) yeniden
  gonderiliyor. Olculmemis ayar (0) GONDERILMEZ
- 0x3E turnikesi karsilastiriliyor, uyusmazlik loglaniyor
- 0x38 ile komut geri bildirimi: olcek ve isaret hatasi arac kimildamadan
  gorulebiliyor
- Port acilamazsa artik sessizce simulasyona dusmuyor, 2 sn'de bir deniyor
- Yapi numarasi karsilastirilmiyor ama DEGISIMI izleniyor

MOD VE E-STOP
- Kip karari kartta (/kart/kip); CH5 esikleme ve debounce kalkti. Kart
  susarsa manuele dusuluyor
- e_stop_node gpio_mod varsayilani False: pin 7'ye bir sey bagli degil ve
  Jetson.GPIO pull_up_down'i yok saydigi icin giris havada kaliyor,
  gurultuyle hayalet E-STOP uretiyor. Gercek kanal 0x34

FREN KIPE BAGLANDI
Kart fren kaynaklarinin buyugunu aliyor ve bizimkini operator cozemiyor.
ackermann_converter hangi kipte oldugunu bilmiyordu: manuelde de fren
hesaplayip basiyordu, yani surucunun gazi biraktigi anda ustune binen ve
acamadigi bir fren. Fren artik tek kapidan (_fren_yayinla) cikiyor ve
manuelde 0 basiyor. E-STOP muaf -- acil durdurma kipten bagimsiz olmali.
Kip bilinmiyor ya da 3 sn'den bayatsa fren SERBEST kaliyor: mod_yoneticisi
otonom kosu ortasinda olurse arac %45 egimde frensiz kalmasin diye.
Manuele gecildigi an bir kez 0 basiliyor -- susmak yetmiyor, kart son
gonderdigimiz degeri tutuyor.

ATIS KILIDI SINIRLANDI
/shoot_command kenar sinyali; True ile False arasinda yayinci olurse fren
kalici basili kaliyor ve her surus komutu sifir hiza cevriliyordu. Arac
bir daha hic hareket etmiyor ve log'a satir dusmuyor. ATIS_AZAMI_S = 12 s
hem ackermann_converter frenine hem seri_kopru hareket kilidine kondu;
sinir dolunca lazer de kapatiliyor.

PANOLAR AYRILDI
Elektrik ekibinin statik panosu 8080'de kaliyor, ROS panosu PANO_PORT'a
(8083) alindi -- iki sunucu ayni portu acamiyor. 3 Eylul'de ROS panosu
kapatilmisti ve gerekcesi o gun DOGRUYDU: kopru /dev/mega ariyordu, arac
alanlari null geliyordu. Kopru 0x30 blogunu konusunca o gerekce kalkiyor;
/kart/* alanlari yalniz o panoda gorunuyor.

DUZELTILEN IKI SESSIZ KUSUR
- gercek_harita ve taret_otonom launch'larinda yinelenen 'baud' anahtari:
  Python sonuncuyu aldigi icin o iki yol 921600 yazilmasina ragmen
  115200'e dusuyordu
- MOD_MANUAL/MOD_FULL_AUTO topics.py'ye tasindi: yayinci ve tuketici ayri
  dugum, iki yerde tutulan sayi ayrisir

NAV2 / KONFIG
- robot_radius yerine gercek footprint (1,90 x 1,16): cevrel yaricap
  1,09 m, 3 m'lik seritte 0,82 m serbest bant birakiyordu
- derinlik kaynaklarinda clearing: false -- gurultulu kaynaga LiDAR'in
  gordugu engeli sildirme yetkisi verilmiyor
- hedefleme_modu: oto; harita modu waypoint'ler bosken kosuyu sessizce
  bitiriyordu
- SLAM /scan/filtered'i okuyor ve minimum_travel_* 0'dan 0,3'e cikti

Mega kalintisi arduino/ agaci silindi. bms_koprusu eklendi (JK BMS ->
/battery/status, olcut bagli degil YAS: BLE kopunca alanlar son degerde
donuyor).

Birim testi 336 -> 601. Yeni denetimlerin hepsi mutasyon turundan gecti:
kaldirilan her dal en az bir testi dusuruyor.

Co-Authored-By: Ahmet Efe Nezli <ahmetefenezli@gmail.com>
Co-Authored-By: Claude Opus 5 <noreply@anthropic.com>
Claude-Session: https://claude.ai/code/session_01DQrHyT88VSwbu22ZNLq7hG

File: urdf/arac.urdf (robot description, URDF)
Before this commit: robot teknofest_ika, 10 links, 9 joints
Links:
- link base_link: geometry collision box size=1.90 1.16 0.76; visual box size=1.90 1.16 0.76

Commit message: fix: kip titremesi, manuel kip hedef iptali, dingil arasi 1.44 ve REEDS_SHEPP
044 ve 047'nin bize dusen maddeleri, 10 Eylul kayan hedef denetimiyle ayni
dosyalarda oldugu icin tek commit'te.

Surus karti arayuzu
  * KIP_TIMEOUT_S 0.5 -> 2.5 s. Esik kopruden gelen tekrar periyodunun
    (DURUM_TAZELEME_S = 1.0) altindaydi; kart kip 2'de sabitken mod saniyede
    iki kez MANUAL<->FULL_AUTO ziplayip her seferinde /mission_start basiyordu,
    misyon FSM'i hic ilerleyemiyordu (sahada olculen: 60 s'de 122 gecis).
  * Kumanda kesmesi (SwA) artik 0.5 s'de bir tekrarlaniyor. Yalniz degisimde
    yayinlanan kesme, acilista e_stop_node ayaga kalkmadan once cikip
    kayboluyordu ve /e_stop false kaliyordu.
  * 0x38 komut karsilastirmasi yalniz otonom kipte. Manuelde kart Jetson
    komutunu tasarim geregi yok sayip kumandadan geleni yolluyor; oradaki
    uyusmazlik uyarisi sahte alarmdi.
  * Kart canliligi /kart/surus'tan olculuyor. /kart/durum|hata|kip onbellekten
    1 Hz tekrarlaniyor, yani hat cop okurken de akiyorlar.
  * F767_TELEMETRI_AKTIF varsayilani 0. Ayni port korumasi zaten vardi;
    varsayilan da kartin tek okuyucusunun seri_kopru oldugunu soylemeli.

Otonomi
  * Manuel kipe gecince ucustaki Nav2 hedefi iptal ediliyor. manual_mod yalniz
    NavigateState.execute girisinde okunuyordu; asama ortasinda SwC otonomdan
    cikarsa hedef ayakta kaliyor ve SwC geri otonoma alindiginda arac bayat bir
    hedefe kalkiyordu. Gorev kaldigi yerden suruyor: asama indeksi ve katedilen
    yol korunuyor, manuel duraklama asama butcesinden sayilmiyor.
  * Planlayici REEDS_SHEPP. DUBIN dar koridorda plan uretemiyor ve hatayi
    yalniz "exceeded maximum iterations" diye veriyor. Arac arkadan kor oldugu
    icin denge reverse_penalty'de: geri yay acik ama pahali, fiilen yalniz
    sikismadan cikarken kullaniliyor. Kayan hedef kapisi geri manevraya
    guvenmiyor, hedefler hala ileride olmak zorunda.
  * Nav2 acilis sonrasi lifecycle dogrulamasi. autostart sabit zaman asimiyla
    dusunce bringup'in tamami iptal oluyor ve bir daha denenmiyor.

Olcumler
  * Dingil arasi 1.40 -> 1.44 (mezurle olculdu, kart ekibiyle teyitli). Deger
    bes yerde yasiyor: ackermann_converter, launch, urdf teker joint'leri
    (+-0.72), nav2_params minimum_turning_radius (2.42 -> 2.49) ve ekf.yaml.
    velocity_smoother acisal tavani 0.37 -> 0.36 (v_max / R_min).
    CAD dogrulama araclari da ayni yaricapa gecti.
    max_steering_angle = 30 derece HALA olculmedi, yer tutucu olarak isaretli.

Kamera ve temizlik
  * Arka kamera konusu /camera/arka/image_raw. Yayinci elektrik tarafinin
    kamera gozcusu ve kamera fisten cikip geri takildiginda cihazi geri baglayan
    da o; ad onunla eslesmek zorunda.
  * Olu on kamera yolu kaldirildi: CAMERA_FRONT_TOPIC'e yayin yapan yoktu,
    /camera_aux/image_processed'i okuyan yoktu.
  * HATA_FREN_STALL pano etiketi "fren ucunda". Bit iki durumu birden
    anlatiyor; serbest yonde stall "fren tam acildi" demek.
  * bms_koprusu'nun rolu aciklandi: BLE'yi okumuyor, :8091'in istemcisi.

Dogrulama
  * Birim testi 804 -> 836, hepsi geciyor. Yeni davranislarin sekizi
    mutasyonla sinandi; ilk yazdigim kart canlilik testi zayifti (adin mesaj
    tipi haritasinda gecmesi yetiyordu), izlenen sozluge daraltildi.
  * scripts/parkur_cad/koridor_dogrula.py kosuldu (kayan hedefin dis
    referansi). Merkez cizgisinin surdugu duz bolumlerde duvara dusen hedef
    3 -> 2; artisin tamami U donuslerinde, orada ic duvar takibi suruyor ve
    duvara temas iki olcumde de 0. Sapma 0.57 / 0.67 m.

Co-Authored-By: Claude Opus 5 <noreply@anthropic.com>
Claude-Session: https://claude.ai/code/session_01AEemac8pGvBbbYhQRaPzic

File: urdf/arac.urdf (robot description, URDF)
Before this commit: robot teknofest_ika, 10 links, 9 joints
Joints:
- joint sag_arka_joint: origin xyz=-0.70 -0.335 -0.10 rpy=0 0 0 -> xyz=-0.72 -0.335 -0.10 rpy=0 0 0
- joint sag_on_joint: origin xyz=0.70 -0.335 -0.10 rpy=0 0 0 -> xyz=0.72 -0.335 -0.10 rpy=0 0 0
- joint sol_arka_joint: origin xyz=-0.70 0.335 -0.10 rpy=0 0 0 -> xyz=-0.72 0.335 -0.10 rpy=0 0 0
- joint sol_on_joint: origin xyz=0.70 0.335 -0.10 rpy=0 0 0 -> xyz=0.72 0.335 -0.10 rpy=0 0 0

Commit message: feat: araçtan olculen govde olculeri koda islendi
Olculen (11 Eylul): en 117 cm · toplam yukseklik 78 cm · dingil arasi 144 cm
(zaten koddaydi) · arka teker merkezleri arasi 100 cm · sasi alti zemin
bosluğu 36,5 cm. Boy bu turda YENIDEN OLCULMEDI, 1,90 kaldi.

EN 1,16 -> 1,17
  nav2 footprint yarim eni 0,580 -> 0,585 (iki costmap), urdf kutusu,
  donus.py'deki CAD araci ve waypoints yorumu birlikte.

IZ GENISLIGI 1,00 m — ILK KEZ OLCULDU
  urdf teker joint'leri y = ±0,335 idi, yani iz 0,67 m. O sayi olculmemisti;
  topics.py'nin kendi yorumu "depoda 0,50 / 0,67 / 0,900 diye uc deger var"
  diyordu. Artik ±0,50.
  Devrilme esikleri YENIDEN HESAPLANDI ama DEGISTIRILMEDI: 1,00 m izle
  statik devrilme acisi agirlik merkezi 0,30-0,60 m icin 59°-40° cikiyor,
  yani koddaki 20°'lik E-STOP esiginin cok ustunde. Esikler §6.5'in zorunlu
  %20 yan egimine (11,31°) gore kurulu, devrilme sinirina gore degil --
  yukseltmek o asamayi riske atar. Gerekce yoruma yazildi.

YUKSEKLIK — yorum farki, ACIKCA belirtiliyor
  78 cm TOPLAM yukseklik kabul edildi, govde kutusunun kendi yuksekligi degil.
  Gerekce: 36,5 + 78 = 114,5 cm olurdu ve bu govdeyi tekerlek capinin ~3 kati
  yapardi; ayrica §7.1 olcu listeleri toplam yuksekligi ister.
  Sonuc: kutu yuksekligi 0,78 - 0,365 = 0,415 m.
  🔑 URDF'te kutu artik ZEMINE DEGMIYOR: sasi alti 0,365 m'de. Eskiden kutu
  zemine oturuyordu ve yuksekligi toplam yukseklik saniliyordu. base_link
  0,28 m'de kaldigi icin kutu merkezi 0,2925 m'ye tasindi.
  ⚠ Bu yorum yanlissa tek satirlik duzeltme.

Dogrulama
  * Birim testi 956 -> 968, hepsi geciyor.
  * URDF'in DUSEY geometrisi artik metin degil ARITMETIK olarak sinaniyor:
    kutu alti = zemin boslugu, kutu ustu = toplam yukseklik, |x| = L/2,
    |y| = iz/2, on tekerler +x arka tekerler -x. XML ayristirilarak.
  * Yedi mutasyonun yedisi yakalandi (eni geri alma, kutuyu toplam yukseklik
    yapma, kutuyu zemine indirme, tek tekerin izini bozma, arka tekeri one
    alma, footprint enini ayristirma, CAD aracini ayristirma).
  * CAD araclari yeniden kosturuldu: U donusleri etkilenmedi (sinir R 4,94 /
    4,81 m). koridor_dogrula: kapsama %61, duvara temas 0, sapma 0,58/0,64 m
    ve 6→7'de hedefsiz 1 -> 0'a dustu. Regresyon yok.

Co-Authored-By: Claude Opus 5 <noreply@anthropic.com>
Claude-Session: https://claude.ai/code/session_01AEemac8pGvBbbYhQRaPzic

File: urdf/arac.urdf (robot description, URDF)
Before this commit: robot teknofest_ika, 10 links, 9 joints
Links:
- link base_link: geometry collision box size=1.90 1.17 0.415; visual box size=1.90 1.17 0.415
Joints:
- joint sag_arka_joint: origin xyz=-0.72 -0.335 -0.10 rpy=0 0 0 -> xyz=-0.72 -0.50 -0.10 rpy=0 0 0
- joint sag_on_joint: origin xyz=0.72 -0.335 -0.10 rpy=0 0 0 -> xyz=0.72 -0.50 -0.10 rpy=0 0 0
- joint sol_arka_joint: origin xyz=-0.72 0.335 -0.10 rpy=0 0 0 -> xyz=-0.72 0.50 -0.10 rpy=0 0 0
- joint sol_on_joint: origin xyz=0.72 0.335 -0.10 rpy=0 0 0 -> xyz=0.72 0.50 -0.10 rpy=0 0 0

Commit message: fix: lidar yuksekligi ZEMIN referansina baglandi (olculen 60 cm)
Olculen: tarama duzlemi zeminden 60 cm.

BULUNAN HATA
LIDAR_Z_M'in yorumu "zeminden tarama duzlemine" diyordu ama sayi dogrudan
base_link'e gore yayinlaniyordu -- hem acilis betiginde hem urdf lidar_joint'te.
base_link zeminden 0,28 m yukarida oldugu icin tarama duzlemi TF'te olculenden
0,28 m DAHA YUKARI yerlesiyordu. Eski deger 0,55 idi, yani TF 0,83 m diyordu.

Bugunku 2B costmap'te etkisi sinirli: `scan` kaynaginda yalnizca
max_obstacle_height: 2.0 var, alt sinir yok, o yuzden nokta filtrelenmiyordu.
Ama sayi yanlisti ve "zeminden" diye olculuyordu -- bir sonraki olcen kisi
ayni hatayi tekrarlardi.

DEGISIKLIK
LIDAR_Z_M artik acikca ZEMINDEN (0.60) ve base_link farki TEK YERDE dusuluyor
(BASE_LINK_Z_M=0.28, urdf base_joint ile ayni). urdf lidar_joint 0.55 -> 0.32.
Acilis betigi hesabi ekrana da basiyor.

⚠ Montaj acisi (yaw) HALA ESKI: 93,3°. LiDAR hub'a tasindigi icin yeniden
kalibre edilmeli (lidar_aci_kalibre.py) -- o aci DORT dugumde kullaniliyor.

YAN DUZELTME
`_urdf_lidar_yaw()` yardimcisi metin deseniyle okuyordu ve joint'in icine bir
yorum eklenince sessizce None donuyordu (bu commit'te tam bu oldu, mevcut test
yakaladi). XML ayristirmaya cevrildi.

Dogrulama
  * Birim testi 968 -> 975, hepsi geciyor.
  * Yeni testler ARITMETIK: urdf'te base_joint + lidar_joint toplami zemin
    yuksekligini vermeli; betikte ham LIDAR_Z_M'in dogrudan TF'e verilmedigi
    ve base_link farkinin dusuldugu ayrica sinaniyor.
  * Uc mutasyonun ucu de yakalandi (lidar_joint'i eskiye dondurme, farki
    dusmeyi kaldirma, eski yuksekligi geri koyma).

Co-Authored-By: Claude Opus 5 <noreply@anthropic.com>
Claude-Session: https://claude.ai/code/session_01AEemac8pGvBbbYhQRaPzic

File: urdf/arac.urdf (robot description, URDF)
Before this commit: robot teknofest_ika, 10 links, 9 joints
Joints:
- joint lidar_joint: origin xyz=0.0 0 0.55 rpy=0 0 1.6284 -> xyz=0.0 0 0.32 rpy=0 0 1.6284

Commit message: feat: govde boyu olculdu (1,83 m) — footprint daraldi
Olculen: toplam boy 183 cm (onceki 1,90 olculmemis bir degerdi).

Tutarlilik: 1,83 - 1,44 (dingil) = 0,39 m toplam tasma. donus.py'nin BAGIMSIZ
arka_tasma=0.20 varsayimi on ucu 0,19 m veriyor -- yani govde aks ortasinda
neredeyse simetrik ve footprint'in +-0,915 simetrigi iyi bir yaklasim.
⚠ Tasmanin one/arkaya dagilimi HALA olculmedi; olculurse footprint'in x
uclari ayri ayri yazilir.

nav2 footprint yari boyu 0,950 -> 0,915 (iki costmap), urdf kutusu, CAD araci
ve test sabiti birlikte.

Dogrulama
  * Birim testi 975/975.
  * Uc mutasyonun ucu yakalandi.
  * koridor_dogrula yeniden kosturuldu, sonuclar asagida degismedi.

Co-Authored-By: Claude Opus 5 <noreply@anthropic.com>
Claude-Session: https://claude.ai/code/session_01AEemac8pGvBbbYhQRaPzic

File: urdf/arac.urdf (robot description, URDF)
Before this commit: robot teknofest_ika, 10 links, 9 joints
Links:
- link base_link: geometry collision box size=1.83 1.17 0.415; visual box size=1.83 1.17 0.415

Commit message: feat: 050/051'den gelen olculer ve SwB gaz tuzagi
Kart ekibinin 050 (olculen degerler) ve 051 (tam arayuz, yapi 15)
belgelerinden koda dusen iki is.

1. TEKERLEK YARICAPI OLCUMDEN TURETILDI — dusey TF zinciri duzeldi
   050 §1: yuvarlanma cevresi 1250 mm olculdu -> r = 1,250/2π = 0,1989 m.
   urdf'te 0,18 yaziliydi ve OLCULMEMISTI; 1,9 cm hata.
   Yaricap base_link'in yuksekligini belirliyor (yaricap + teker joint ofseti
   0,10), o da ZEMINDEN olculen her seyin base_link'e gore ofsetini belirliyor.
   Zincir yeniden hesaplandi:
     base_joint   0.28   -> 0.2989
     govde kutusu 0.2925 -> 0.2736   (alti hala zeminden 0,365 m)
     lidar_joint  0.32   -> 0.3011   (tarama duzlemi hala zeminden 0,60 m)
     teker silindiri yaricapi 0.18 -> 0.1989
   BASE_LINK_Z_M acilis betiginde de guncellendi; test ikisinin ayni oldugunu
   ve zeminden olculen degerlerin korundugunu ARITMETIKLE dogruluyor.

2. 🔴 SwB YUKARIDAYKEN OTONOMDA GAZ YOK — artik soyleniyor
   051 §6.3: kart taret kipini ROLANTI kumesine koyuyor ve bu kural OTONOMDA
   DA gecerli. Fren ve direksiyon etkilenmiyor, yani belirti "direksiyon
   donuyor ama arac kimildamiyor" ve sebebi hicbir logda yoktu -- bit panoda
   yalnizca 'taret' diye gorunuyor, gazla iliskisi gorunmuyor.
   seri_kopru artik OTONOM kipte DRM_TARET kalkikken acik bir hata satiri
   basiyor. Manuelde basilmiyor: orada SwB'yi kaldirmak normal bir is.

Dogrulama
  * Birim testi 975 -> 984, hepsi geciyor.
  * Dort mutasyonun dordu yakalandi.

Co-Authored-By: Claude Opus 5 <noreply@anthropic.com>
Claude-Session: https://claude.ai/code/session_01AEemac8pGvBbbYhQRaPzic

File: urdf/arac.urdf (robot description, URDF)
Before this commit: robot teknofest_ika, 10 links, 9 joints
Links:
- link sag_arka_teker: geometry collision cylinder length=0.15 radius=0.1989; visual cylinder length=0.15 radius=0.1989
- link sag_on_teker: geometry collision cylinder length=0.15 radius=0.1989; visual cylinder length=0.15 radius=0.1989
- link sol_arka_teker: geometry collision cylinder length=0.15 radius=0.1989; visual cylinder length=0.15 radius=0.1989
- link sol_on_teker: geometry collision cylinder length=0.15 radius=0.1989; visual cylinder length=0.15 radius=0.1989
Joints:
- joint base_joint: origin xyz=0 0 0.28 rpy=0 0 0 -> xyz=0 0 0.2989 rpy=0 0 0
- joint lidar_joint: origin xyz=0.0 0 0.32 rpy=0 0 1.6284 -> xyz=0.0 0 0.3011 rpy=0 0 1.6284
